Commit message: !

File: URDF/ABOT/urdf/ABOT.urdf (robot description, URDF)
Before this commit: robot ABOT, 4 links, 3 joints
Links:
- removed link base_link
- added link abot_base, mass 0.274585554808092; collision mesh filename=package://abot/meshes/abot_base.STL; visual mesh filename=package://abot/meshes/abot_base.STL
- link abot_caster_wheel: geometry collision mesh filename=package://abot/meshes/abot_caster_wheel.STL; visual mesh filename=package://abot/meshes/abot_caster_wheel.STL
- link abot_left_wheel: geometry collision mesh filename=package://abot/meshes/abot_left_wheel.STL; visual mesh filename=package://abot/meshes/abot_left_wheel.STL
- link abot_right_wheel: geometry collision mesh filename=package://abot/meshes/abot_right_wheel.STL; visual mesh filename=package://abot/meshes/abot_right_wheel.STL
Joints:
- joint caster_wheel_to_base: origin xyz=0 0.078 -0.011 rpy=0 0 -1.5707963267949 -> xyz=-0.078 0 -0.011 rpy=0 0 0; parent base_link -> abot_base
- joint left_wheel_to_base: origin xyz=0.068 0 0.0145 rpy=0 -0.1987 -1.5708 -> xyz=0 0.068 0.0145 rpy=0 -0.1987 0; parent base_link -> abot_base
- joint right_wheel_to_base: origin xyz=-0.068 0 0.0145 rpy=0 0 -1.5708 -> xyz=0 -0.068 0.0145 rpy=0 0 0; parent base_link -> abot_base

Commit message: !

File: URDF/ABOT/urdf/ABOT.urdf (robot description, URDF)
Before this commit: robot abot, 4 links, 3 joints
Links:
- link abot_base: mass 0.274585554808092 -> 0.27459
- link abot_caster_wheel: mass 0 -> 0.011207
- link abot_right_wheel: mass 0.0504636002883635 -> 0.050464
Joints:
- joint left_wheel_to_base: origin xyz=0 0.068 0.0145 rpy=0 -0.1987 0 -> xyz=0 0.068 0.0145 rpy=0 0 0

Commit message: !

File: URDF/ABOT/urdf/ABOT.urdf (robot description, URDF)
Before this commit: robot abot, 4 links, 3 joints
Links:
- link abot_base: mass 0.27459 -> 0.390932406092716
- link abot_caster_wheel: mass 0.011207 -> 0.0112066893138855
- link abot_right_wheel: mass 0.050464 -> 0.0504636002883635
Joints:
- joint caster_wheel_to_base: axis 0 0 0 -> 0 1 0

Commit message: !

File: URDF/ABOT/urdf/ABOT.urdf (robot description, URDF)
Before this commit: robot abot, 4 links, 3 joints
Links:
- added link abot_lidar, mass 0; collision mesh filename=package://abot/meshes/abot_lidar.STL; visual mesh filename=package://abot/meshes/abot_lidar.STL
- link abot_base: mass 0.390932406092716 -> 0.537364562401972
- link abot_caster_wheel: mass 0.0112066893138855 -> 0.011207
- link abot_left_wheel: mass 0.050464 -> 0.0504636002883634
Joints:
- added joint lidar_to_base: type fixed, parent abot_base, child abot_lidar, origin xyz=-0.01 0 0.1319 rpy=0 0 3.1416, axis 0 0 0
- joint caster_wheel_to_base: axis 0 1 0 -> 0 0 0
- joint right_wheel_to_base: origin xyz=0 -0.068 0.0145 rpy=0 0 0 -> xyz=0 -0.0680000000000001 0.0144999999999995 rpy=0 0 0

Commit message: !

File: URDF/ABOT/urdf/ABOT.urdf (robot description, URDF)
Before this commit: robot abot, 5 links, 4 joints
Links:
- link abot_base: mass 0.537364562401972 -> 0.54627
- link abot_caster_wheel: mass 0.011207 -> 0.0112066893138855
- link abot_left_wheel: mass 0.0504636002883634 -> 0.050464
Joints:
- joint caster_wheel_to_base: axis 0 0 0 -> 0 1 0
- joint lidar_to_base: origin xyz=-0.01 0 0.1319 rpy=0 0 3.1416 -> xyz=-0.0100000000000004 0 0.1419 rpy=0 0 3.14159265358978
- joint right_wheel_to_base: origin xyz=0 -0.0680000000000001 0.0144999999999995 rpy=0 0 0 -> xyz=0 -0.068 0.0145 rpy=0 0 0
